File: Hardware/Design Files/[02] - TOP.kicad_sch (KiCad schematic)
At the start: 0 parts

Commit message: first commit after nas abckup;
Parts:
- added FID1, FID2, FID3: Fiducial, Miscellaneous:FID, symbol Mechanical:Fiducial
- added H1, H2, H3, H4: MountingHole, MountingHole:MountingHole_3.5mm_Pad_Via, symbol Mechanical:MountingHole
- added H5, H6, H7, H8: MountingHole_Pad, MountingHole:MountingHole_2.7mm_Pad, symbol Mechanical:MountingHole_Pad
Connections:
- new net +12V: H7.1
- new net +VDC: H5.1
- new net GND: H6.1, H8.1
Other:
- sheet MCU ports: added 3V3_PGOOD, I2C1_SCL, I2C1_SDA, MCU_NRST, MCU_SWCLK, MCU_SWDIO, MCU_USART1_RX, MCU_USART1_TX, PA0, PA1, QUADSPI_BK1_IO0, QUADSPI_BK1_IO1, QUADSPI_BK1_IO2, QUADSPI_BK1_IO3, QUADSPI_BK1_NCS, QUADSPI_CLK, TIM1_CH1, TIM2_CH1, TIM2_CH2, USBD_N, USBD_P; removed none
- sheet MEM ports: added SCLK, SI/SIO0, SO/SIO1, nCS, nRST/SIO3, nWP/SIO2; removed none
- sheet POWER ports: added 12V_PGOOD; removed none
- sheet UI ports: added 12V_PGOOD, 3V3_PGOOD, LED_B, LED_G, LED_R, OLED_SCL, OLED_SDA, OLED_nRST, PB1, PB2, TC_NRST, TC_SW_CLK, TC_SW_DIO, TC_UART_RX, TC_UART_TX, USBD_N, USBD_P; removed none
