File: Hardware/Design Files/[03] - POWER.kicad_sch (KiCad schematic)
At the start: 45 parts, among them Q1 FDMS86550, Q2 FDMS86550, Q3 FDMS86550, Q4 FDMS86550, U1 LM34936-Q1

Commit message: first commit after nas abckup;
Parts:
- added C33, C46, C47, C48: 10uF, Capacitor_SMD:C_1206_3216Metric, symbol Device:C
- added C34, C49: 68uF, Capacitor_SMD:CP_Elec_10x10, symbol Device:C_Polarized
- added C44, C45: 4.7uF, Capacitor_SMD:C_1206_3216Metric, symbol Device:C
- added R20: 10K, Resistor_SMD:R_0603_1608Metric, symbol Device:R
- C10, C20, C21: renamed from C?; footprint (none) -> Capacitor_SMD:C_0603_1608Metric; Part Number (none) -> CL10B104KB8NNNC
- C11: renamed from C?; footprint (none) -> Capacitor_SMD:C_0805_2012Metric; Part Number (none) -> CL21A475KAQNNNE
- C12, C18, C19, C6: renamed from C?; footprint (none) -> Capacitor_SMD:C_0603_1608Metric; Part Number (none) -> CL10C101JB8NNNC
- C13: renamed from C?; footprint (none) -> Capacitor_SMD:CP_Elec_10x10
- C14, C7: renamed from C?; footprint (none) -> Capacitor_SMD:C_0603_1608Metric; Part Number (none) -> CL10B223KB8WPNC
- C15, C16, C17: renamed from C?; footprint (none) -> Capacitor_SMD:C_0603_1608Metric; Part Number (none) -> CL10C470JB8NNNC
- C22, C24, C25: renamed from C?; footprint (none) -> Capacitor_SMD:C_1206_3216Metric; Part Number (none) -> CL31A106MBHNNNE
- C23: renamed from C?; footprint (none) -> Capacitor_SMD:C_0603_1608Metric; Part Number (none) -> CL10B105KP8NNNC
- C8, C9: renamed from C?; footprint (none) -> Capacitor_SMD:C_1206_3216Metric; Part Number (none) -> CL31A475KBHNNNE
- D1, D4: renamed from D?; footprint (none) -> Diode_SMD:D_SMC
- L1: renamed from L?; footprint (none) -> Inductors:IND_SER20xx
- Q1, Q2, Q3, Q4: Part Number (none) -> FDMS86540
- R10, R13, R15, R9: renamed from R?; footprint (none) -> Resistor_SMD:R_0603_1608Metric; Part Number (none) -> RC0603FR-0710RL
- R11, R12, R7, R8: renamed from R?; footprint (none) -> Resistor_SMD:R_0603_1608Metric; Part Number (none) -> RC0603FR-07100RL
- R14: renamed from R?; value R -> 8mR; footprint (none) -> Resistors:RES_3015-WIDE
- R16: renamed from R?; value 0R -> 8mR; footprint (none) -> Resistors:RES_3015-WIDE
- R2, R3, R4: renamed from R?; footprint (none) -> Resistor_SMD:R_0603_1608Metric; Part Number (none) -> RC0603FR-0727K4L
- R5: renamed from R?; footprint (none) -> Resistor_SMD:R_0603_1608Metric; Part Number (none) -> RC0603FR-0710KL
- R6: renamed from R?; footprint (none) -> Resistor_SMD:R_0603_1608Metric; Part Number (none) -> RT0603BRD0793K1L
- U1: Part Number (none) -> LM34936-Q1
- gave numbers to parts that had none: 2
Connections:
- net +12V: now also C33.1, C34.1, C49.1
- net +VDC: now also C44.2, C45.2
- net 12V_ISNSP: now also C46.1, C47.1, C48.1
- net 12V_PGOOD: now also R20.2
- net 12V_RT: no longer C6.2, U1.4 (SLOPE)
- net GND: now also C33.2, C34.2, C44.1, C45.1, C46.2, C47.2, C48.2, C49.2
- net VCC: now also R20.1
- new net 12V_SLOPE: C6.2, U1.4 (SLOPE)
Other:
- note added: "PLACE C23 NEAR PIN 21"
- note removed: "PLACE C? NEAR PIN 24"
- moved on the sheet: C11, C13, C18, C19, C20, C21, C22, C23, C24, C25, C6, C8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
