File: Hardware/Design Files/[04] - MCU.kicad_sch (KiCad schematic)
At the start: 8 parts, among them U2 STM32L432KCUx

Commit message: first commit after nas abckup;
Parts:
- added C35, C36: 4.7uF, Capacitor_SMD:C_0805_2012Metric, symbol Device:C
- added C39, C40, C41, C42: 0.1uF, Capacitor_SMD:C_0603_1608Metric, symbol Device:C
- added L2: 2.2uH, Inductors:WE-XHMA, symbol Device:L
- added R21, R22, R28, R29, R30, R31, R32, R34, R35: R, Resistor_SMD:R_0603_1608Metric, symbol Device:R
- added U3: TPS62150, Package_DFN_QFN:VQFN-16-1EP_3x3mm_P0.5mm_EP1.68x1.68mm, symbol Regulator_Switching:TPS62150
- added U5: LM393, Package_SO:SOIC-8_3.9x4.9mm_P1.27mm, symbol Comparator:LM393
- C1: footprint (none) -> Capacitor_SMD:C_0805_2012Metric; Part Number (none) -> CL21A475KAQNNNE
- C2, C3: footprint (none) -> Capacitor_SMD:C_0603_1608Metric; Part Number (none) -> CL10B105KP8NNNC
- C4, C5: value 100nF -> 0.1uF; footprint (none) -> Capacitor_SMD:C_0603_1608Metric; Part Number (none) -> CL10B104KB8NNNC
- C43: renamed from C10n1; footprint (none) -> Capacitor_SMD:C_0603_1608Metric; Part Number (none) -> CL10B103KB8NNNC
- R1: footprint (none) -> Resistor_SMD:R_0603_1608Metric
- U2: Part Number (none) -> STM32L432KCU6
Connections:
- net +3.3V: now also C36.1, C42.1, L2.2, R21.1, R32.1, R34.1, R35.1, U3.14 (VOS), U5.8 (V+)
- net GND: now also U2.16 (VSS), U2.32 (VSS), U2.33 (VSS), C35.2, C36.2, C39.2, C40.2, C41.2, C42.2, R22.2, R29.2, R31.2, U3.15 (PGND), U3.16 (PGND), U3.17 (EP), U3.6 (AGND), U3.7 (FSW), U3.8 (DEF), U5.4 (V-)
- net ADC1_IN9: now reaches U2.10 (PA4)
- net ADC1_IN9: now also C39.1, U5.1, U5.2 (-)
- net ADC1_IN10: now reaches U2.11 (PA5)
- net ADC1_IN10: now also C40.1, U5.6 (-), U5.7
- net QUADSPI_BK1_IO3: now reaches U2.12 (PA6)
- net QUADSPI_BK1_IO2: now reaches U2.13 (PA7)
- net QUADSPI_BK1_IO1: now reaches U2.14 (PB0)
- net QUADSPI_BK1_IO0: now reaches U2.15 (PB1)
- net TIM1_CH1: now reaches U2.18 (PA8)
- net MCU_USART1_TX: now reaches U2.19 (PA9)
- net MCU_USART1_RX: now reaches U2.20 (PA10)
- net USBD_N: now reaches U2.21 (PA11)
- net USBD_P: now reaches U2.22 (PA12)
- net MCU_SWDIO: now reaches U2.23 (PA13)
- net MCU_SWCLK: now reaches U2.24 (PA14)
- net TIM2_CH1: now reaches U2.25 (PA15)
- net TIM2_CH2: now reaches U2.26 (PB3)
- net 3V3_PGOOD: now reaches U2.27 (PB4)
- net 3V3_PGOOD: now also R32.2, U3.4 (PG)
- net I2C1_SCL: now reaches U2.29 (PB6)
- net I2C1_SCL: now also R35.2
- net I2C1_SDA: now reaches U2.30 (PB7)
- net I2C1_SDA: now also R34.2
- net PA0: now reaches U2.6 (PA0)
- net PA1: now reaches U2.7 (PA1)
- net QUADSPI_BK1_NCS: now reaches U2.8 (PA2)
- net QUADSPI_CLK: now reaches U2.9 (PA3)
- new net: R30.2, R31.1, U5.5 (+)
- new net: R28.2, R29.1, U5.3 (+)
- new net: C41.1, U3.9 (SS/TR)
- new net: L2.1, U3.1 (SW), U3.2 (SW), U3.3 (SW)
- new net: R21.2, R22.1, U3.5 (FB)
- new net +12V: C35.1, R30.1, U3.10 (AVIN), U3.11 (PVIN), U3.12 (PVIN), U3.13 (EN)
- new net +VDC: R28.1
- no-connect marks 0 -> 3
