File: Hardware/Design Files/[05] - MEM.kicad_sch (KiCad schematic)
At the start: 0 parts

Commit message: first commit after nas abckup;
Parts:
- added C38: 0.1uF, Capacitor_SMD:C_0603_1608Metric, symbol Device:C
- added U4: MX25R3235FZNxx0, Package_SON:WSON-8-1EP_6x5mm_P1.27mm_EP3.4x4mm, symbol Memory_Flash:MX25R3235FZNxx0
Connections:
- new net +3.3V: C38.1, U4.8 (VCC)
- new net GND: C38.2, U4.4 (GND), U4.9 (GND)
- new net SCLK: U4.6 (SCLK)
- new net SI/SIO0: U4.5 (SI/SIO0)
- new net SO/SIO1: U4.2 (SO/SIO1)
- new net nCS: U4.1 (~{CS})
- new net nRST/SIO3: U4.7 (~{RESET}/SIO3)
- new net nWP/SIO2: U4.3 (~{WP}/SIO2)
Changed lines of the file:
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@@
 (kicad_sch (version 20211123) (generator eeschema)
   (paper "A4")
+  (wire (pts (xy 147.32 92.075) (xy 140.97 92.075))
+    (stroke (width 0) (type default) (color 0 0 0 0))
+  )
+  (wire (pts (xy 110.49 89.535) (xy 115.57 89.535))
+    (stroke (width 0) (type default) (color 0 0 0 0))
+  )
+  (wire (pts (xy 110.49 97.155) (xy 115.57 97.155))
+    (stroke (width 0) (type default) (color 0 0 0 0))
+  )
+  (wire (pts (xy 110.49 94.615) (xy 115.57 94.615))
+    (stroke (width 0) (type default) (color 0 0 0 0))
+  )
+  (wire (pts (xy 183.515 82.55) (xy 183.515 85.09))
+    (stroke (width 0) (type default) (color 0 0 0 0))
+  )
+  (wire (pts (xy 110.49 86.995) (xy 115.57 86.995))
+    (stroke (width 0) (type default) (color 0 0 0 0))
+  )
+  (wire (pts (xy 110.49 92.075) (xy 115.57 92.075))
+    (stroke (width 0) (type default) (color 0 0 0 0))
+  )
+  (wire (pts (xy 183.515 92.71) (xy 183.515 95.25))
+    (stroke (width 0) (type default) (color 0 0 0 0))
+  )
+  (hierarchical_label "SI{slash}SIO0" (shape bidirectional) (at 110.49 86.995 180)
+    (effects (font (size 1.27 1.27)) (justify right))
+  )
+  (hierarchical_label "SO{slash}SIO1" (shape bidirectional) (at 147.32 92.075 0)
+    (effects (font (size 1.27 1.27)) (justify left))
+  )
+  (hierarchical_label "SCLK" (shape output) (at 110.49 89.535 180)
+    (effects (font (size 1.27 1.27)) (justify right))
+  )
+  (hierarchical_label "nRST{slash}SIO3" (shape bidirectional) (at 110.49 97.155 180)
+    (effects (font (size 1.27 1.27)) (justify right))
+  )
+  (hierarchical_label "nCS" (shape output) (at 110.49 92.075 180)
+    (effects (font (size 1.27 1.27)) (justify right))
+  )
+  (hierarchical_label "nWP{slash}SIO2" (shape bidirectional) (at 110.49 94.615 180)
+    (effects (font (size 1.27 1.27)) (justify right))
+  )
+  (symbol (lib_id "Memory_Flash:MX25R3235FZNxx0") (at 128.27 92.075 0) (unit 1)
+    (in_bom yes) (on_board yes)
+    (property "Reference" "U4" (id 0) (at 136.525 100.965 0))
+    (property "Value" "MX25R3235FZNxx0" (id 1) (at 120.015 100.965 0))
+    (property "Footprint" "Package_SON:WSON-8-1EP_6x5mm_P1.27mm_EP3.4x4mm" (id 2) (at 128.27 107.315 0)
+      (effects (font (size 1.27 1.27)) hide)
+    )
+    (property "Datasheet" "http://www.macronix.com/Lists/Datasheet/Attachments/7534/MX25R3235F,%20Wide%20Range,%2032Mb,%20v1.6.pdf" (id 3) (at 128.27 92.075 0)
+      (effects (font (size 1.27 1.27)) hide)
+    )
+    (property "Part Number" "MX25R3235FZNIL0" (id 4) (at 128.27 92.075 0)
+      (effects (font (size 1.27 1.27)) hide)
+    )
+    (pin "1")
+    (pin "2")
+    (pin "3")
+    (pin "4")
+    (pin "5")
+    (pin "6")
+    (pin "7")
+    (pin "8")
+    (pin "9")
+  )
+  (symbol (lib_id "power:+3.3V") (at 183.515 82.55 0) (unit 1)
+    (in_bom yes) (on_board yes) (fields_autoplaced)
+    (property "Reference" "#PWR050" (id 0) (at 183.515 86.36 0)
+      (effects (font (size 1.27 1.27)) hide)
+    )
+    (property "Value" "+3.3V" (id 1) (at 183.515 77.47 0))
+    (property "Footprint" "" (id 2) (at 183.515 82.55 0)
+      (effects (font (size 1.27 1.27)) hide)
+    )
+    (property "Datasheet" "" (id 3) (at 183.515 82.55 0)
+      (effects (font (size 1.27 1.27)) hide)
+    )
+    (pin "1")
+  )
+  (symbol (lib_id "power:GND") (at 133.35 102.235 0) (unit 1)
+    (in_bom yes) (on_board yes) (fields_autoplaced)
+    (property "Reference" "#PWR049" (id 0) (at 133.35 108.585 0)
+      (effects (font (size 1.27 1.27)) hide)
+    )
+    (property "Value" "GND" (id 1) (at 133.35 107.315 0))
+    (property "Footprint" "" (id 2) (at 133.35 102.235 0)
+      (effects (font (size 1.27 1.27)) hide)
+    )
+    (property "Datasheet" "" (id 3) (at 133.35 102.235 0)
+      (effects (font (size 1.27 1.27)) hide)
+    )
+    (pin "1")
+  )
+  (symbol (lib_id "power:+3.3V") (at 133.35 81.915 0) (unit 1)
+    (in_bom yes) (on_board yes) (fields_autoplaced)
+    (property "Reference" "#PWR048" (id 0) (at 133.35 85.725 0)
+      (effects (font (size 1.27 1.27)) hide)
+    )
+    (property "Value" "+3.3V" (id 1) (at 133.35 76.835 0))
+    (property "Footprint" "" (id 2) (at 133.35 81.915 0)
+      (effects (font (size 1.27 1.27)) hide)
+    )
+    (property "Datasheet" "" (id 3) (at 133.35 81.915 0)
+      (effects (font (size 1.27 1.27)) hide)
+    )
+    (pin "1")
+  )
+  (symbol (lib_id "Device:C") (at 183.515 88.9 0) (unit 1)
+    (in_bom yes) (on_board yes) (fields_autoplaced)
+    (property "Reference" "C38" (id 0) (at 187.325 87.6299 0)
+      (effects (font (size 1.27 1.27)) (justify left))
+    )
+    (property "Value" "0.1uF" (id 1) (at 187.325 90.1699 0)
+      (effects (font (size 1.27 1.27)) (justify left))
+    )
+    (property "Footprint" "Capacitor_SMD:C_0603_1608Metric" (id 2) (at 184.4802 92.71 0)
+      (effects (font (size 1.27 1.27)) hide)
+    )
+    (property "Datasheet" "~" (id 3) (at 183.515 88.9 0)
+      (effects (font (size 1.27 1.27)) hide)
+    )
+    (property "Part Number" "CL10B104KB8NNNC" (id 4) (at 183.515 88.9 0)
+      (effects (font (size 1.27 1.27)) hide)
+    )
+    (pin "1")
+    (pin "2")
+  )
+  (symbol (lib_id "power:GND") (at 183.515 95.25 0) (unit 1)
+    (in_bom yes) (on_board yes) (fields_autoplaced)
+    (property "Reference" "#PWR051" (id 0) (at 183.515 101.6 0)
+      (effects (font (size 1.27 1.27)) hide)
+    )
+    (property "Value" "GND" (id 1) (at 183.515 100.33 0))
+    (property "Footprint" "" (id 2) (at 183.515 95.25 0)
+      (effects (font (size 1.27 1.27)) hide)
+    )
+    (property "Datasheet" "" (id 3) (at 183.515 95.25 0)
+      (effects (font (size 1.27 1.27)) hide)
+    )
+    (pin "1")
+  )
 )
