File: Hardware/Design Files/[06] - UI.kicad_sch (KiCad schematic)
At the start: 0 parts

Commit message: first commit after nas abckup;
Parts:
- added C26, C27, C28, C31, C32, C37: 1uF, Capacitor_SMD:C_0603_1608Metric, symbol Device:C
- added C29: 4.7uF, Capacitor_SMD:C_0603_1608Metric, symbol Device:C
- added C30: 2.2uF, Capacitor_SMD:C_0603_1608Metric, symbol Device:C
- added D5, D6, D8: LED, LED_SMD:LED_0603_1608Metric, symbol Device:LED
- added D7: LED_RGBA, Diodes:LTST-C19HE1WT, symbol Device:LED_RGBA
- added J1: 0541043031, Connectors:0541043031, symbol Connectors:0541043031
- added J2: USB_C_Receptacle, Connector_USB:USB_C_Receptacle_Molex_105450-0101, symbol Connector:USB_C_Receptacle
- added J3: TC2050, Connector:Tag-Connect_TC2050-IDC-FP_2x05_P1.27mm_Vertical, symbol Miscellaneous:TC2050
- added R17, R18, R23, R24, R33: 10K, Resistor_SMD:R_0603_1608Metric, symbol Device:R
- added R19: 390K, Resistor_SMD:R_0603_1608Metric, symbol Device:R
- added R25, R26, R27: 100R, Resistor_SMD:R_0603_1608Metric, symbol Device:R
- added SW1, SW2: SW_Push, Button_Switch_SMD:SW_Push_1P1T_NO_Vertical_Wuerth_434133025816, symbol Switch:SW_Push
Connections:
- new net: C30.1, J1.27
- new net: D6.1 (K), R24.1
- new net: J1.26, R19.1
- new net: D8.1 (K), R33.1
- new net: D7.2 (GK), R26.2
- new net: C32.1, J1.5
- new net: C32.2, J1.4
- new net: D5.1 (K), R23.1
- new net: J2.A4 (VBUS), J2.A9 (VBUS), J2.B4 (VBUS), J2.B9 (VBUS)
- new net: J2.A5 (CC1), R18.2
- new net: J2.B5 (CC2), R17.1
- new net: D7.3 (BK), R27.2
- new net: C31.1, J1.3
- new net: C31.2, J1.2
- new net: C29.1, J1.28
- new net: D7.1 (RK), R25.2
- new net +3.3V: C27.2, C28.2, D5.2 (A), J1.11, J1.6, J1.9, J3.1
- new net 12V_PGOOD: D6.2 (A)
- new net 3V3_PGOOD: D8.2 (A)
- new net GND: C26.1, C27.1, C28.1, C29.2, C30.2, C37.1, D7.4 (A), J1.1, J1.10, J1.12, J1.13, J1.15, J1.16, J1.17, J1.21, J1.22, J1.23, J1.24, J1.25, J1.29, J1.30, J1.8, J2.A1 (GND), J2.A12 (GND), J2.B1 (GND), J2.B12 (GND), J2.S1 (SHIELD), J3.9, R17.2, R18.1, R19.2, R23.2, R24.2, R33.2, SW1.2, SW2.2
- new net LED_B: R27.1
- new net LED_G: R26.1
- new net LED_R: R25.1
- new net OLED_SCL: J1.18
- new net OLED_SDA: J1.19, J1.20
- new net OLED_nRST: J1.14
- new net PB1: C37.2, SW1.1
- new net PB2: C26.2, SW2.1
- new net TC_NRST: J3.7
- new net TC_SW_CLK: J3.5
- new net TC_SW_DIO: J3.3
- new net TC_UART_RX: J3.2
- new net TC_UART_TX: J3.4
- new net USBD_N: J2.A7 (D-), J2.B7 (D-)
- new net USBD_P: J2.A6 (D+), J2.B6 (D+)
- no-connect marks 0 -> 15
